File: 2_boardSystem/eagle-brd/V2/ScoreBoard-V2/ScoreBoard-V2.brd (EAGLE design)
At the start: 196.2 x 89.8 mm, 44 parts, among them M1 VNH5019, M2 VNH5019, M3 VNH5019, M4 VNH5019, M5 VNH5019, M6 VNH5019, U1 TXB0108PWR

Commit message: board v2 work in progress
Parts:
- removed PW$1: DC/DC-STEP-DOWNGLOB, diy-modules:DC/DC-STEP-DOWN-UNIVERSAL
- added D1: ES2D, diode:SMB
- added SP-DW: DC/DC-STEP-DOWNGLOB, diy-modules:DC/DC-STEP-DOWN-UNIVERSAL
- moved SJ2 2.37 mm to (55.9, 79.8), turned to 180 degrees
- moved MOT-P 2.29 mm to (2.54, 64.5)
- moved C1 2.16 mm to (3.17, 46.7)
- moved ARDUINO_MEGA_1 0.38 mm to (187.3, 105.2)
- moved C2 0.38 mm to (184.2, 82.9)
- moved C3 0.38 mm to (131.4, 83.6)
- moved D-SUB50 0.38 mm to (94.0, 77.2)
- moved F1 0.38 mm to (103.5, 56.3)
- moved F2 0.38 mm to (103.5, 22.0)
- moved F3 0.38 mm to (61.6, 56.3)
- moved F4 0.38 mm to (61.6, 22.0)
- moved F5 0.38 mm to (20.3, 56.3)
- moved F6 0.38 mm to (20.3, 22.0)
- moved FAN-PWR 0.38 mm to (2.54, 34.0)
- moved H2 0.38 mm to (4.45, 85.5)
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Connections:
- new net N$2: D1.A, MOT-P.1
- net GND: now also SP-DW.OUT-, SP-DW.OUT-1, SP-DW.OUT-2; no longer PW$1.OUT-, PW$1.OUT-1, PW$1.OUT-2
- net GNDA: now also SP-DW.IN-, SP-DW.IN-1, SP-DW.IN-2; no longer PW$1.IN-, PW$1.IN-1, PW$1.IN-2
- net N$4: now also SP-DW.OUT+, SP-DW.OUT+1, SP-DW.OUT+2; no longer PW$1.OUT+, PW$1.OUT+1, PW$1.OUT+2
- net V+: now also SP-DW.IN+, SP-DW.IN+1, SP-DW.IN+2; no longer PW$1.IN+, PW$1.IN+1, PW$1.IN+2
- net VDD: now also D1.C; no longer MOT-P.1
Routing:
- net +5V: track 419.1 -> 487.5 mm, vias 3 -> 4
- net N$4: track 25.0 -> 43.8 mm
- net N$2: track 0.00 -> 5.88 mm
- net IN3B: track 94.0 -> 96.2 mm
- net VDD: track 247.7 -> 249.3 mm
- net M3-: track 41.2 -> 42.7 mm
- net N$1: track 14.9 -> 16.3 mm
- net M4-: track 82.0 -> 83.2 mm
- net IM5V: track 150.2 -> 151.1 mm
- net IM3V: track 118.0 -> 117.1 mm
- net V+: track 46.4 -> 45.6 mm
- net M1+: track 74.4 -> 75.0 mm
- net RP-SCK: track 47.5 -> 48.1 mm
- net M5+: track 91.0 -> 91.6 mm
- net IN4B: track 70.5 -> 71.0 mm
Other:
- board text added: "Com-enable"
