File: 2_boardSystem/V2/HW/ScoreBoard-V2/ScoreBoard-V2.sch (EAGLE design)
At the start: 43 parts, among them M1 VNH5019, M2 VNH5019, M3 VNH5019, M4 VNH5019, M5 VNH5019, M6 VNH5019, U1 TXB0108

Commit message: license and library
Parts:
- added V-OFF-PAD, V-REF-PAD: TP2P2-38-17, testpad:TP2P2-38-17
Connections:
- net GND: now also V-OFF-PADB.TP, V-REF-PADB.TP
- net V-OFF: now also V-OFF-PADA.TP
- net V-REF: now also V-REF-PADA.TP
Other:
- moved on the sheet: ARDUINO_MEGA_1, C2, R-REF, RESET-LOGIC

Commit message: ScorBoard-manual-V2
Parts:
- added AREF-JP: (no value), jumper:JP1E
- added COM-EN: PTR1PAD1-13, testpad:PTR1PAD1-13
Connections:
- new net V-REF-TRIMM: AREF-JP.2, R-REF.S, V-REF-PADA.TP
- net COM-ENABLE: now also COM-EN.TP
- net V-REF: now also AREF-JP.1; no longer R-REF.S, V-REF-PADA.TP
Other:
- moved on the sheet: C2, V-REF-PADA
Changed lines of the file:
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@@
 <attribute name="SPICEPREFIX" value="X"/>
 </part>
+<part name="AREF-JP" library="jumper" library_urn="urn:adsk.eagle:library:252" deviceset="JP1E" device="" package3d_urn="urn:adsk.eagle:package:15455/1"/>
+<part name="COM-EN" library="testpad" deviceset="PTR1" device="PAD1-13" package3d_urn="urn:adsk.eagle:package:27946/1"/>
 </parts>
 <sheets>
@@
 <wire x1="140.97" y1="35.56" x2="78.74" y2="35.56" width="0.1524" layer="94"/>
 <wire x1="78.74" y1="35.56" x2="78.74" y2="91.44" width="0.1524" layer="94"/>
-<text x="80.01" y="81.28" size="1.016" layer="97">Pull OE low to place all
+<text x="80.01" y="85.09" size="1.016" layer="97">Pull OE low to place all
 outputs in 3-state mode.</text>
 <wire x1="156.845" y1="95.25" x2="154.305" y2="95.25" width="0.1524" layer="97"/>
@@
 <text x="50.8" y="160.02" size="1.27" layer="97">Solder when voltage
 is calibrated</text>
-<text x="171.45" y="161.29" size="1.016" layer="97">I 3.3V del mega sono stabilizzati dai 5V che gli entrano.
+<text x="170.18" y="162.56" size="1.016" layer="97">I 3.3V del mega sono stabilizzati dai 5V che gli entrano.
 Se come unico carico viene messo un partitore, l'uscita
 sarà molto stabile e adatta a essere usata come Aref.
@@
 motori alla lettura dell'ADC.
 La precisione è fondamentale</text>
-<text x="171.45" y="147.32" size="1.016" layer="97">I VNH5019 hanno sul CS un uscita di 140mV/A.
+<text x="181.61" y="147.32" size="1.016" layer="97">I VNH5019 hanno sul CS un uscita di 140mV/A.
 Imax 1A    --&gt; V-ref=140mV
 Imax 1.5A --&gt; V-ref=210mV
@@
 <instance part="R-REF" gate="G$1" x="152.4" y="163.83" smashed="yes">
 <attribute name="NAME" x="148.971" y="160.02" size="1.778" layer="95" rot="R90"/>
-<attribute name="VALUE" x="154.94" y="166.37" size="1.778" layer="96" rot="R90"/>
+<attribute name="VALUE" x="148.59" y="167.64" size="1.778" layer="96"/>
 </instance>
 <instance part="GND7" gate="1" x="152.4" y="151.13" smashed="yes">
 <attribute name="VALUE" x="149.86" y="148.59" size="1.778" layer="96"/>
 </instance>
-<instance part="C2" gate="G$1" x="158.75" y="160.02" smashed="yes" rot="MR0">
-<attribute name="NAME" x="157.226" y="160.401" size="1.778" layer="95" rot="MR0"/>
-<attribute name="VALUE" x="157.226" y="155.321" size="1.778" layer="96" rot="MR0"/>
+<instance part="C2" gate="G$1" x="161.29" y="160.02" smashed="yes" rot="MR0">
+<attribute name="NAME" x="159.766" y="160.401" size="1.778" layer="95" rot="MR0"/>
+<attribute name="VALUE" x="159.766" y="155.321" size="1.778" layer="96" rot="MR0"/>
 </instance>
 <instance part="VDD11" gate="G$1" x="52.07" y="144.78" smashed="yes">
@@
 </instance>
 <instance part="V-OFF-PAD" gate="A" x="233.68" y="167.64" smashed="yes">
-<attribute name="NAME" x="229.87" y="168.91" size="1.778" layer="95"/>
+<attribute name="NAME" x="224.79" y="168.91" size="1.778" layer="95"/>
 <attribute name="TP_SIGNAL_NAME" x="234.95" y="166.37" size="1.778" layer="97"/>
 </instance>
@@
 <attribute name="TP_SIGNAL_NAME" x="232.41" y="152.4" size="1.778" layer="97" rot="R180"/>
 </instance>
-<instance part="V-REF-PAD" gate="A" x="161.29" y="167.64" smashed="yes">
-<attribute name="NAME" x="157.48" y="167.64" size="1.4224" layer="95"/>
-<attribute name="TP_SIGNAL_NAME" x="162.56" y="166.37" size="1.778" layer="97"/>
+<instance part="V-REF-PAD" gate="A" x="158.75" y="167.64" smashed="yes">
+<attribute name="NAME" x="155.575" y="168.275" size="0.8128" layer="95"/>
+<attribute name="TP_SIGNAL_NAME" x="160.02" y="166.37" size="1.778" layer="97"/>
 </instance>
 <instance part="V-REF-PAD" gate="B" x="161.29" y="151.13" smashed="yes" rot="R180">
-<attribute name="NAME" x="157.48" y="148.59" size="1.4224" layer="95"/>
+<attribute name="NAME" x="158.115" y="149.86" size="0.8128" layer="95"/>
 <attribute name="TP_SIGNAL_NAME" x="160.02" y="152.4" size="1.778" layer="97" rot="R180"/>
+</instance>
+<instance part="AREF-JP" gate="A" x="166.37" y="166.37" smashed="yes" rot="MR0">
+<attribute name="NAME" x="168.91" y="170.18" size="1.4224" layer="95" rot="MR270"/>
+<attribute name="VALUE" x="160.655" y="166.37" size="1.778" layer="96" rot="MR90"/>
+</instance>
+<instance part="COM-EN" gate="G$1" x="91.44" y="81.28" smashed="yes" rot="R270">
+<attribute name="NAME" x="85.09" y="82.296" size="1.27" layer="95"/>
+<attribute name="TP_SIGNAL_NAME" x="88.9" y="80.01" size="1.778" layer="97" rot="R270"/>
 </instance>
 </instances>
@@
 <pinref part="C2" gate="G$1" pin="2"/>
 <wire x1="152.4" y1="154.94" x2="152.4" y2="158.75" width="0.1524" layer="91"/>
-<wire x1="158.75" y1="154.94" x2="152.4" y2="154.94" width="0.1524" layer="91"/>
+<wire x1="161.29" y1="154.94" x2="152.4" y2="154.94" width="0.1524" layer="91"/>
 <junction x="152.4" y="154.94"/>
 <pinref part="V-REF-PAD" gate="B" pin="TP"/>
-<wire x1="158.75" y1="154.94" x2="161.29" y2="154.94" width="0.1524" layer="91"/>
 <wire x1="161.29" y1="154.94" x2="161.29" y2="153.67" width="0.1524" layer="91"/>
-<junction x="158.75" y="154.94"/>
+<junction x="161.29" y="154.94"/>
 </segment>
 <segment>
@@
 <pinref part="U1" gate="G$1" pin="OE"/>
 <wire x1="95.25" y1="78.74" x2="93.98" y2="78.74" width="0.1524" layer="91"/>
-<label x="93.98" y="78.74" size="1.27" layer="95" rot="R180" xref="yes"/>
+<label x="92.71" y="78.74" size="1.27" layer="95" rot="R180" xref="yes"/>
+<pinref part="COM-EN" gate="G$1" pin="TP"/>
+<wire x1="93.98" y1="78.74" x2="92.71" y2="78.74" width="0.1524" layer="91"/>
+<wire x1="93.98" y1="81.28" x2="93.98" y2="78.74" width="0.1524" layer="91"/>
+<junction x="93.98" y="78.74"/>
 </segment>
 <segment>
@@
 <net name="V-REF" class="4">
 <segment>
-<pinref part="R-REF" gate="G$1" pin="S"/>
-<label x="170.18" y="163.83" size="1.27" layer="95" rot="MR0" xref="yes"/>
-<wire x1="157.48" y1="163.83" x2="158.75" y2="163.83" width="0.1524" layer="91"/>
-<pinref part="C2" gate="G$1" pin="1"/>
-<wire x1="158.75" y1="163.83" x2="158.75" y2="162.56" width="0.1524" layer="91"/>
-<junction x="158.75" y="163.83"/>
-<wire x1="158.75" y1="163.83" x2="161.29" y2="163.83" width="0.1524" layer="91"/>
-<pinref part="V-REF-PAD" gate="A" pin="TP"/>
-<wire x1="161.29" y1="163.83" x2="162.56" y2="163.83" width="0.1524" layer="91"/>
-<wire x1="161.29" y1="165.1" x2="161.29" y2="163.83" width="0.1524" layer="91"/>
-<junction x="161.29" y="163.83"/>
-</segment>
-<segment>
 <label x="162.56" y="118.11" size="1.27" layer="95" rot="MR0" xref="yes"/>
 <wire x1="162.56" y1="118.11" x2="165.1" y2="118.11" width="0.1524" layer="91"/>
 <pinref part="ARDUINO_MEGA_1" gate="G$1" pin="AREF"/>
+</segment>
+<segment>
+<pinref part="AREF-JP" gate="A" pin="1"/>
+<wire x1="166.37" y1="163.83" x2="166.37" y2="162.56" width="0.1524" layer="91"/>
+<label x="175.26" y="158.75" size="1.016" layer="95" rot="R180" xref="yes"/>
+<wire x1="166.37" y1="162.56" x2="166.37" y2="158.75" width="0.1524" layer="91"/>
+<wire x1="166.37" y1="158.75" x2="168.91" y2="158.75" width="0.1524" layer="91"/>
+<pinref part="C2" gate="G$1" pin="1"/>
+<wire x1="161.29" y1="162.56" x2="166.37" y2="162.56" width="0.1524" layer="91"/>
+<junction x="166.37" y="162.56"/>
 </segment>
 </net>
@@
 <net name="V-OFF" class="4">
 <segment>
+<pinref part="ARDUINO_MEGA_1" gate="G$1" pin="A01(PF1/ADC1)"/>
+<wire x1="165.1" y1="113.03" x2="162.56" y2="113.03" width="0.1524" layer="91"/>
+<label x="162.56" y="113.03" size="1.016" layer="95" rot="R180" xref="yes"/>
+</segment>
+<segment>
+<label x="242.57" y="163.83" size="1.016" layer="95" rot="R180" xref="yes"/>
 <pinref part="R-OFF" gate="G$1" pin="S"/>
 <wire x1="224.79" y1="163.83" x2="226.06" y2="163.83" width="0.1524" layer="91"/>
 <pinref part="C3" gate="G$1" pin="1"/>
 <wire x1="226.06" y1="163.83" x2="233.68" y2="163.83" width="0.1524" layer="91"/>
-<wire x1="233.68" y1="163.83" x2="238.76" y2="163.83" width="0.1524" layer="91"/>
+<wire x1="233.68" y1="163.83" x2="236.22" y2="163.83" width="0.1524" layer="91"/>
 <wire x1="226.06" y1="163.83" x2="226.06" y2="162.56" width="0.1524" layer="91"/>
 <junction x="226.06" y="163.83"/>
-<label x="245.11" y="163.83" size="1.016" layer="95" rot="R180" xref="yes"/>
 <pinref part="V-OFF-PAD" gate="A" pin="TP"/>
 <wire x1="233.68" y1="165.1" x2="233.68" y2="163.83" width="0.1524" layer="91"/>
 <junction x="233.68" y="163.83"/>
 </segment>
-<segment>
-<pinref part="ARDUINO_MEGA_1" gate="G$1" pin="A01(PF1/ADC1)"/>
-<wire x1="165.1" y1="113.03" x2="162.56" y2="113.03" width="0.1524" layer="91"/>
-<label x="162.56" y="113.03" size="1.016" layer="95" rot="R180" xref="yes"/>
-</segment>
 </net>
 <net name="N$2" class="1">
@@
 </segment>
 </net>
+<net name="V-REF-TRIMM" class="4">
+<segment>
+<pinref part="R-REF" gate="G$1" pin="S"/>
+<wire x1="157.48" y1="163.83" x2="158.75" y2="163.83" width="0.1524" layer="91"/>
+<junction x="158.75" y="163.83"/>
+<pinref part="V-REF-PAD" gate="A" pin="TP"/>
+<wire x1="158.75" y1="165.1" x2="158.75" y2="163.83" width="0.1524" layer="91"/>
+<junction x="158.75" y="163.83"/>
+<pinref part="AREF-JP" gate="A" pin="2"/>
+<wire x1="163.83" y1="163.83" x2="158.75" y2="163.83" width="0.1524" layer="91"/>
+</segment>
+</net>

Commit message: ScorBoard-manual-V2
Parts:
- removed D1: ES2D, diode:ES2D
Connections:
- removed net N$2: D1.A, MOT-SW-1.KL
- net VDD: now also MOT-SW-1.KL; no longer D1.C
Changed lines of the file:
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@@
 <part name="U$1" library="loghi" deviceset="ALFY-BIG" device=""/>
 <part name="U$4" library="loghi" deviceset="ALFY-BIG" device=""/>
-<part name="D1" library="diode" library_urn="urn:adsk.eagle:library:210" deviceset="ES2D" device="" package3d_urn="urn:adsk.eagle:package:43404/2"/>
 <part name="V-OFF-PAD" library="testpad" deviceset="TP2" device="P2-38-17" package3d_urn="urn:adsk.eagle:package:27945/1">
 <attribute name="SPICEPREFIX" value="X"/>
@@
 </instance>
 <instance part="U$1" gate="G$1" x="10.16" y="15.24" smashed="yes"/>
-<instance part="D1" gate="G$1" x="22.86" y="138.43" smashed="yes" rot="MR180">
-<attribute name="NAME" x="21.59" y="136.6774" size="1.778" layer="95" rot="MR180"/>
-</instance>
 <instance part="V-OFF-PAD" gate="A" x="233.68" y="167.64" smashed="yes">
 <attribute name="NAME" x="224.79" y="168.91" size="1.778" layer="95"/>
@@
 <pinref part="C1" gate="G$1" pin="+"/>
 <wire x1="27.94" y1="138.43" x2="30.48" y2="138.43" width="0.1524" layer="91"/>
-<pinref part="D1" gate="G$1" pin="C"/>
-<wire x1="25.4" y1="138.43" x2="27.94" y2="138.43" width="0.1524" layer="91"/>
 <junction x="27.94" y="138.43"/>
+<pinref part="MOT-SW" gate="-1" pin="KL"/>
+<wire x1="17.78" y1="138.43" x2="27.94" y2="138.43" width="0.1524" layer="91"/>
 </segment>
 <segment>
@@
 </segment>
 </net>
-<net name="N$2" class="1">
-<segment>
-<pinref part="D1" gate="G$1" pin="A"/>
-<pinref part="MOT-SW" gate="-1" pin="KL"/>
-<wire x1="20.32" y1="138.43" x2="17.78" y2="138.43" width="0.1524" layer="91"/>
-</segment>
-</net>
