File: 2_boardSystem/V2/HW/ScoreBoard-V2/ScoreBoard-V2.brd (EAGLE design)
At the start: 196.2 x 89.8 mm, 45 parts, among them M1 VNH5019, M2 VNH5019, M3 VNH5019, M4 VNH5019, M5 VNH5019, M6 VNH5019, U1 TXB0108

Commit message: license and library
Parts:
- added V-OFF-PAD, V-REF-PAD: TP2P2-38-17, testpad:P2-38-17
Connections:
- net GND: now also V-OFF-PAD.TP-2, V-REF-PAD.TP-2
- net V-OFF: now also V-OFF-PAD.TP-1
- net V-REF: now also V-REF-PAD.TP-1
Routing:
- net V-REF: track 64.2 -> 98.8 mm
- net GND: track 519.8 -> 544.3 mm
- net V-OFF: track 77.3 -> 79.9 mm
- net CHA2: track 130.9 -> 132.0 mm
Changed lines of the file:
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@@
 <attribute name="MF" value="" x="46.99" y="112.776" size="1.778" layer="27" rot="R180" display="off"/>
 <attribute name="MPN" value="" x="46.99" y="112.776" size="1.778" layer="27" rot="R180" display="off"/>
-<attribute name="NAME" x="89.535" y="86.106" size="1.778" layer="25" ratio="10" rot="SR0"/>
+<attribute name="NAME" x="84.455" y="86.106" size="1.778" layer="25" ratio="10" rot="SR0"/>
 <attribute name="OC_FARNELL" value="unknown" x="46.99" y="112.776" size="1.778" layer="27" rot="R180" display="off"/>
 <attribute name="OC_NEWARK" value="unknown" x="46.99" y="112.776" size="1.778" layer="27" rot="R180" display="off"/>
@@
 <attribute name="VALUE" x="55.4799" y="79.756" size="0.02" layer="27" rot="R180"/>
 </element>
-<element name="VTEST-" library="testpad" library_urn="urn:adsk.eagle:library:385" package="P2-38-17" package3d_urn="urn:adsk.eagle:package:27945/1" value="TP2P2-38-17" x="55.88" y="72.136" smashed="yes" rot="R270">
+<element name="VTEST-" library="testpad" package="P2-38-17" package3d_urn="urn:adsk.eagle:package:27945/1" value="TP2P2-38-17" x="55.88" y="72.136" smashed="yes" rot="R270">
 <attribute name="SPICEPREFIX" value="X" x="24.13" y="31.496" size="1.778" layer="27" rot="R270" display="off"/>
 <attribute name="TP_SIGNAL_NAME" value="" x="50.165" y="74.676" size="1" layer="37" rot="R270"/>
@@
 <element name="D1" library="diode" library_urn="urn:adsk.eagle:library:210" package="SMB" package3d_urn="urn:adsk.eagle:package:43404/2" value="ES2D" x="5.715" y="56.261" smashed="yes" rot="R180">
 <attribute name="NAME" x="8.001" y="57.785" size="1.27" layer="25"/>
+</element>
+<element name="V-OFF-PAD" library="testpad" package="P2-38-17" package3d_urn="urn:adsk.eagle:package:27945/1" value="TP2P2-38-17" x="128.27" y="86.995" smashed="yes" rot="R180">
+<attribute name="NAME" x="124.46" y="87.63" size="1.27" layer="25" ratio="10" rot="R180"/>
+<attribute name="SPICEPREFIX" value="X" x="128.27" y="86.995" size="1.778" layer="27" rot="R180" display="off"/>
+<attribute name="TP_SIGNAL_NAME" value="" x="128.27" y="86.995" size="1.778" layer="27" rot="R180" display="off"/>
+</element>
+<element name="V-REF-PAD" library="testpad" package="P2-38-17" package3d_urn="urn:adsk.eagle:package:27945/1" value="TP2P2-38-17" x="111.125" y="86.995" smashed="yes" rot="R180">
+<attribute name="NAME" x="107.315" y="87.63" size="1.27" layer="25" ratio="10" rot="R180"/>
+<attribute name="SPICEPREFIX" value="X" x="111.125" y="86.995" size="1.778" layer="27" rot="R180" display="off"/>
+<attribute name="TP_SIGNAL_NAME" value="" x="111.125" y="86.995" size="1.778" layer="27" rot="R180" display="off"/>
 </element>
 </elements>
@@
 <wire x1="191.135" y1="70.866" x2="191.77" y2="70.231" width="0.4064" layer="16"/>
 <wire x1="191.77" y1="70.231" x2="191.77" y2="69.596" width="0.4064" layer="16"/>
+<contactref element="V-OFF-PAD" pad="TP-2"/>
+<contactref element="V-REF-PAD" pad="TP-2"/>
+<wire x1="126.365" y1="86.995" x2="129.794" y2="83.566" width="0.2032" layer="16"/>
+<wire x1="129.794" y1="83.566" x2="130.175" y2="83.566" width="0.2032" layer="16"/>
+<wire x1="109.22" y1="86.995" x2="111.76" y2="84.455" width="0.2032" layer="1"/>
+<wire x1="123.825" y1="84.455" x2="126.365" y2="86.995" width="0.2032" layer="1"/>
+<wire x1="111.76" y1="84.455" x2="123.825" y2="84.455" width="0.2032" layer="1"/>
 </signal>
 <signal name="+5V" class="3">
@@
 <contactref element="D-SUB50" pad="1"/>
 <contactref element="ARDUINO_MEGA_1" pad="A9"/>
-<wire x1="123.66625" y1="87.53475" x2="116.205" y2="80.0735" width="0.1524" layer="16"/>
-<wire x1="182.88" y1="87.53475" x2="123.66625" y2="87.53475" width="0.1524" layer="16"/>
+<wire x1="116.205" y1="80.0735" x2="123.66625" y2="87.53475" width="0.1524" layer="16"/>
 <wire x1="182.88" y1="58.4835" x2="182.88" y2="87.53475" width="0.1524" layer="16"/>
 <wire x1="186.69" y1="54.6735" x2="182.88" y2="58.4835" width="0.1524" layer="16"/>
@@
 <wire x1="184.785" y1="28.956" x2="186.69" y2="30.861" width="0.1524" layer="16"/>
 <wire x1="116.205" y1="80.0735" x2="116.0526" y2="80.0608" width="0.1524" layer="16"/>
+<wire x1="123.66625" y1="87.53475" x2="123.825" y2="87.53475" width="0.1524" layer="16"/>
+<wire x1="135.89" y1="87.53475" x2="182.88" y2="87.53475" width="0.1524" layer="16"/>
+<wire x1="123.825" y1="87.53475" x2="125.19025" y2="88.9" width="0.1524" layer="16"/>
+<wire x1="134.52475" y1="88.9" x2="135.89" y2="87.53475" width="0.1524" layer="16"/>
+<wire x1="125.19025" y1="88.9" x2="134.52475" y2="88.9" width="0.1524" layer="16"/>
 </signal>
 <signal name="CHA1" class="4">
@@
 <wire x1="184.15" y1="84.201" x2="187.16625" y2="81.18475" width="0.1524" layer="16"/>
 <wire x1="137.00125" y1="81.50225" x2="136.525" y2="81.026" width="0.1524" layer="1"/>
-<wire x1="181.45125" y1="81.50225" x2="137.00125" y2="81.50225" width="0.1524" layer="1"/>
+<wire x1="181.45125" y1="81.50225" x2="140.97" y2="81.50225" width="0.1524" layer="1"/>
+<wire x1="140.97" y1="81.50225" x2="137.00125" y2="81.50225" width="0.1524" layer="1"/>
 <wire x1="184.15" y1="84.201" x2="181.45125" y2="81.50225" width="0.1524" layer="1"/>
+<contactref element="V-REF-PAD" pad="TP-1"/>
+<wire x1="113.03" y1="86.995" x2="123.19" y2="86.995" width="0.2032" layer="1"/>
+<wire x1="123.19" y1="86.995" x2="125.095" y2="88.9" width="0.2032" layer="1"/>
+<wire x1="125.095" y1="88.9" x2="138.43" y2="88.9" width="0.2032" layer="1"/>
+<wire x1="140.97" y1="86.36" x2="140.97" y2="81.50225" width="0.2032" layer="1"/>
+<wire x1="138.43" y1="88.9" x2="140.97" y2="86.36" width="0.2032" layer="1"/>
 </signal>
 <signal name="N$5">
@@
 <wire x1="132.715" y1="87.21725" x2="149.38375" y2="87.21725" width="0.1524" layer="16"/>
 <wire x1="132.715" y1="83.566" x2="132.715" y2="87.21725" width="0.1524" layer="16"/>
+<contactref element="V-OFF-PAD" pad="TP-1"/>
+<wire x1="130.175" y1="86.995" x2="130.39725" y2="87.21725" width="0.1524" layer="16"/>
+<wire x1="130.39725" y1="87.21725" x2="132.715" y2="87.21725" width="0.1524" layer="16"/>
 </signal>
 <signal name="M3-FUSE" class="1">

Commit message: ScorBoard-manual-V2
Parts:
- added AREF-JP: (no value), jumper:JP1
- added COM-EN: PTR1PAD1-13, testpad:P1-13
Connections:
- new net V-REF-TRIMM: AREF-JP.2, R-REF.2, V-REF-PAD.TP-1
- net COM-ENABLE: now also COM-EN.TP
- net V-REF: now also AREF-JP.1; no longer R-REF.2, V-REF-PAD.TP-1
Routing:
- net V-REF-TRIMM: track 0.00 -> 90.0 mm, vias 0 -> 1
- net V-REF: track 98.8 -> 71.9 mm
- net GND: track 544.3 -> 553.7 mm
- net V-OFF: track 79.9 -> 75.9 mm
- net CHA2: track 132.0 -> 129.8 mm
- net COM-ENABLE: track 29.4 -> 30.5 mm
Other:
- board text removed: "Com-enable"

Commit message: ScorBoard-manual-V2
Parts:
- removed D1: ES2D, diode:SMB
Connections:
- removed net N$2: D1.A, MOT-SW.1
- net VDD: now also MOT-SW.1; no longer D1.C
Routing:
- net GNDA: track 291.2 -> 284.1 mm
- net VDD: track 252.5 -> 258.9 mm
- net N$2: track 5.88 -> 0.00 mm
- net V-OFF: track 75.9 -> 79.9 mm
- net V-REF: track 71.9 -> 71.2 mm
Changed lines of the file:
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@@
 <drawing>
 <settings>
-<setting alwaysvectorfont="yes"/>
+<setting alwaysvectorfont="no"/>
 <setting verticaltext="up"/>
 </settings>
@@
 <element name="U$2" library="loghi" package="ALFY_15MM" value="" x="4.445" y="18.161" smashed="yes"/>
 <element name="U$3" library="loghi" package="ALFY_15MM" value="" x="116.205" y="48.006" smashed="yes" rot="MR0"/>
-<element name="D1" library="diode" library_urn="urn:adsk.eagle:library:210" package="SMB" package3d_urn="urn:adsk.eagle:package:43404/2" value="ES2D" x="5.715" y="56.261" smashed="yes" rot="R180">
-<attribute name="NAME" x="8.001" y="57.785" size="1.27" layer="25"/>
-</element>
 <element name="V-OFF-PAD" library="testpad" package="P2-38-17" package3d_urn="urn:adsk.eagle:package:27945/1" value="TP2P2-38-17" x="128.27" y="86.995" smashed="yes" rot="R180">
 <attribute name="NAME" x="125.095" y="88.265" size="1.016" layer="25" ratio="10"/>
@@
 <wire x1="12.85875" y1="54.991" x2="12.7" y2="54.991" width="1.778" layer="1"/>
 <wire x1="12.85875" y1="54.991" x2="13.335" y2="54.356" width="1.778" layer="1"/>
-<wire x1="3.175" y1="44.196" x2="3.175" y2="44.831" width="1.778" layer="1"/>
-<wire x1="15.71625" y1="65.786" x2="11.7475" y2="69.75475" width="1.778" layer="16"/>
 <wire x1="11.7475" y1="69.75475" x2="11.303" y2="70.485" width="1.778" layer="16"/>
-<wire x1="3.81" y1="36.536" x2="4.32625" y2="37.05225" width="2.54" layer="1"/>
 <wire x1="3.81" y1="36.536" x2="3.175" y2="37.171" width="2.54" layer="1"/>
 <wire x1="3.175" y1="37.171" x2="3.175" y2="44.196" width="2.54" layer="1"/>
@@
 <wire x1="16.51" y1="37.39589375" x2="8.382" y2="29.26789375" width="2.54" layer="16"/>
 <wire x1="16.619" y1="37.16125" x2="16.619" y2="37.50489375" width="1.778" layer="16"/>
-<wire x1="16.619" y1="37.16125" x2="16.51" y2="37.05225" width="1.778" layer="16"/>
 <wire x1="3.81" y1="36.536" x2="11.771" y2="36.536" width="2.54" layer="1"/>
 <wire x1="11.771" y1="36.536" x2="13.335" y2="38.1" width="2.54" layer="1"/>
@@
 <wire x1="53.18125" y1="72.136" x2="63.34125" y2="72.136" width="0.635" layer="1"/>
 <wire x1="52.3875" y1="72.92975" x2="53.18125" y2="72.136" width="0.635" layer="1"/>
-<wire x1="44.1325" y1="72.92975" x2="52.3875" y2="72.92975" width="0.635" layer="1"/>
-<wire x1="15.5575" y1="44.35475" x2="44.1325" y2="72.92975" width="0.635" layer="1"/>
-<wire x1="13.49375" y1="44.35475" x2="15.5575" y2="44.35475" width="0.635" layer="1"/>
+<wire x1="48.5775" y1="72.92975" x2="52.3875" y2="72.92975" width="0.635" layer="1"/>
+<wire x1="20.0025" y1="44.35475" x2="48.5775" y2="72.92975" width="0.635" layer="1"/>
+<wire x1="13.49375" y1="44.35475" x2="20.0025" y2="44.35475" width="0.635" layer="1"/>
 <wire x1="13.49375" y1="44.35475" x2="13.335" y2="44.196" width="0.635" layer="1"/>
 <wire x1="67.865625" y1="76.660375" x2="67.865625" y2="79.041625" width="0.635" layer="1"/>
@@
 <wire x1="3.81" y1="31.496" x2="24.13" y2="31.496" width="2.54" layer="1"/>
 <wire x1="3.81" y1="31.496" x2="3.81" y2="31.536" width="2.54" layer="1"/>
-<wire x1="24.13" y1="56.896" x2="20.32" y2="53.086" width="2.54" layer="1"/>
-<wire x1="24.13" y1="64.516" x2="24.13" y2="56.896" width="2.54" layer="1"/>
-<wire x1="24.13" y1="64.516" x2="10.16" y2="64.516" width="2.54" layer="1"/>
+<wire x1="26.035" y1="56.261" x2="22.86" y2="53.086" width="2.54" layer="1"/>
+<wire x1="22.86" y1="53.086" x2="20.32" y2="53.086" width="2.54" layer="1"/>
+<wire x1="26.035" y1="64.516" x2="26.035" y2="56.261" width="2.54" layer="1"/>
+<wire x1="26.035" y1="64.516" x2="10.16" y2="64.516" width="2.54" layer="1"/>
 <wire x1="24.92375" y1="31.8135" x2="27.14625" y2="34.036" width="2.54" layer="1"/>
 <wire x1="24.92375" y1="31.8135" x2="24.13" y2="31.496" width="1.778" layer="1"/>
-<contactref element="D1" pad="C"/>
-<wire x1="7.915" y1="56.261" x2="7.915" y2="62.271" width="2.54" layer="1"/>
-<wire x1="7.915" y1="62.271" x2="10.16" y2="64.516" width="2.54" layer="1"/>
-<wire x1="3.175" y1="49.276" x2="3.175" y2="50.378" width="2.54" layer="1"/>
-<wire x1="7.915" y1="55.118" x2="7.915" y2="56.261" width="2.54" layer="1"/>
-<wire x1="7.915" y1="55.118" x2="3.175" y2="50.378" width="2.54" layer="1"/>
 <wire x1="101.981" y1="34.036" x2="103.505" y2="35.56" width="2.54" layer="1"/>
 <via x="103.505" y="35.56" extent="1-16" drill="1.016"/>
@@
 <wire x1="61.595" y1="18.796" x2="61.595" y2="21.971" width="1.778" layer="1"/>
 <via x="61.595" y="21.971" extent="1-16" drill="1.016"/>
+<contactref element="MOT-SW" pad="1"/>
+<wire x1="7.66" y1="62.016" x2="3.81" y2="62.016" width="2.54" layer="1"/>
+<wire x1="10.16" y1="64.516" x2="7.66" y2="62.016" width="2.54" layer="1"/>
+<wire x1="3.81" y1="62.016" x2="3.81" y2="52.07" width="2.54" layer="1"/>
+<wire x1="3.81" y1="52.07" x2="3.175" y2="51.435" width="2.54" layer="1"/>
+<wire x1="3.175" y1="51.435" x2="3.175" y2="49.276" width="2.54" layer="1"/>
 </signal>
 <signal name="PWM1" class="4">
@@
 <signal name="V-REF" class="4">
 <contactref element="ARDUINO_MEGA_1" pad="AREF"/>
-<wire x1="137.00125" y1="81.50225" x2="136.525" y2="81.026" width="0.1524" layer="1"/>
 <contactref element="AREF-JP" pad="1"/>
 <wire x1="120.65" y1="86.995" x2="121.92" y2="86.995" width="0.2032" layer="1"/>
@@
 <signal name="V-OFF" class="4">
 <contactref element="ARDUINO_MEGA_1" pad="A1"/>
-<wire x1="149.38375" y1="87.21725" x2="184.785" y2="51.816" width="0.1524" layer="16"/>
-<wire x1="132.715" y1="87.21725" x2="149.38375" y2="87.21725" width="0.1524" layer="16"/>
-<wire x1="130.39725" y1="87.21725" x2="132.715" y2="87.21725" width="0.1524" layer="16"/>
+<wire x1="184.785" y1="51.816" x2="149.38375" y2="87.21725" width="0.1524" layer="16"/>
 <contactref element="R-OFF" pad="2"/>
 <contactref element="C3" pad="1"/>
@@
 <wire x1="132.715" y1="78.486" x2="131.445" y2="77.216" width="0.1524" layer="16"/>
 <wire x1="132.715" y1="83.566" x2="132.715" y2="78.486" width="0.1524" layer="16"/>
-<wire x1="130.175" y1="86.995" x2="130.39725" y2="87.21725" width="0" layer="19" extent="16-16"/>
-<wire x1="132.715" y1="83.566" x2="132.715" y2="87.21725" width="0" layer="19" extent="16-16"/>
+<wire x1="130.39725" y1="87.21725" x2="130.175" y2="86.995" width="0.1524" layer="16"/>
+<wire x1="149.38375" y1="87.21725" x2="132.715" y2="87.21725" width="0.1524" layer="16"/>
+<wire x1="132.715" y1="87.21725" x2="130.39725" y2="87.21725" width="0.1524" layer="16"/>
+<wire x1="132.715" y1="83.566" x2="132.715" y2="87.21725" width="0.1524" layer="16"/>
 </signal>
 <signal name="M3-FUSE" class="1">
@@
 <wire x1="13.335" y1="25.146" x2="20.32" y2="25.146" width="1.778" layer="1"/>
 </signal>
-<signal name="N$2" class="1">
-<contactref element="D1" pad="A"/>
-<contactref element="MOT-SW" pad="1"/>
-<wire x1="3.81" y1="62.016" x2="3.81" y2="56.556" width="2.54" layer="1"/>
-<wire x1="3.81" y1="56.556" x2="3.515" y2="56.261" width="2.54" layer="1"/>
-</signal>
 <signal name="V-REF-TRIMM" class="4">

Commit message: ScorBoard-manual-V2
Routing:
- net GND: track 553.7 -> 597.0 mm
- net +5V: track 487.5 -> 496.5 mm, vias 4 -> 6
- net IM4V: track 108.4 -> 116.9 mm
- net M3-: track 42.7 -> 44.6 mm
- net AR-SCK: track 44.4 -> 46.2 mm
- net AR-ATX/PRX: track 37.7 -> 39.4 mm
- net AR-MISO: track 37.9 -> 39.1 mm
- net GNDA: track 284.1 -> 282.9 mm
- net RP-SCK: track 48.1 -> 49.1 mm
- net N$1: track 16.3 -> 17.0 mm
- net PWM4: track 83.2 -> 82.7 mm
- net COM-ENABLE: track 30.5 -> 31.0 mm
